File: hardware/3D-tracker.brd (EAGLE design)
At the start: 63.2 x 47 mm, 24 parts, among them IC1 TS4231, IC2 NRF52840, IC3 MIC5233-3.3YS, Q1 DMP2035U

Commit message: Update electrical scheme, add gerber file, add hw images
Parts:
- R2: value 470R -> 15R
- R3: value 15R -> 470R
Connections:
- net N$14 renamed P1.13
- net N$2 renamed P1.11
- net N$4 renamed P1.10
- net N$5 renamed P0.03
Changed lines of the file:
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@@
 <attribute name="VALUE" x="22.86" y="19.685" size="1.27" layer="27" rot="R270"/>
 </element>
-<element name="R2" library="resistor" library_urn="urn:adsk.eagle:library:348" package="R0805" package3d_urn="urn:adsk.eagle:package:23553/2" value="470R" x="60.96" y="34.29" smashed="yes" rot="R270">
+<element name="R2" library="resistor" library_urn="urn:adsk.eagle:library:348" package="R0805" package3d_urn="urn:adsk.eagle:package:23553/2" value="15R" x="60.96" y="34.29" smashed="yes" rot="R270">
 <attribute name="NAME" x="59.944" y="36.322" size="1.27" layer="25"/>
 <attribute name="VALUE" x="58.42" y="34.925" size="1.27" layer="27" rot="R270"/>
 </element>
-<element name="R3" library="resistor" library_urn="urn:adsk.eagle:library:348" package="R0805" package3d_urn="urn:adsk.eagle:package:23553/2" value="15R" x="58.42" y="34.29" smashed="yes" rot="R270">
+<element name="R3" library="resistor" library_urn="urn:adsk.eagle:library:348" package="R0805" package3d_urn="urn:adsk.eagle:package:23553/2" value="470R" x="58.42" y="34.29" smashed="yes" rot="R270">
 <attribute name="NAME" x="57.404" y="36.322" size="1.27" layer="25"/>
 <attribute name="VALUE" x="55.88" y="34.925" size="1.27" layer="27" rot="R270"/>
@@
 <wire x1="30.099" y1="13.97" x2="30.099" y2="11.7095625" width="0.254" layer="1"/>
 <wire x1="30.099" y1="13.97" x2="30.099" y2="14.859" width="0.1524" layer="1"/>
-<wire x1="42.545" y1="10.16" x2="41.91" y2="9.525" width="0" layer="19" extent="1-1"/>
+<wire x1="42.545" y1="10.16" x2="41.91" y2="10.16" width="0" layer="19" extent="1-1"/>
 </signal>
 <signal name="SWC">
@@
 <wire x1="21.59" y1="12.7" x2="21.59" y2="12.192" width="0.4064" layer="1"/>
 </signal>
-<signal name="N$2">
+<signal name="P1.11">
 <contactref element="IC2" pad="1"/>
 <contactref element="R2" pad="2"/>
@@
 <wire x1="60.96" y1="31.75" x2="60.96" y2="33.34" width="0.254" layer="1"/>
 </signal>
-<signal name="N$4">
+<signal name="P1.10">
 <contactref element="IC2" pad="2"/>
 <contactref element="R3" pad="2"/>
@@
 <wire x1="58.42" y1="32.131" x2="58.42" y2="33.34" width="0.254" layer="1"/>
 </signal>
-<signal name="N$5">
+<signal name="P0.03">
 <contactref element="IC2" pad="3"/>
 <contactref element="R4" pad="2"/>
@@
 <wire x1="52.49" y1="8.8764" x2="52.4764" y2="8.89" width="0.254" layer="1"/>
 </signal>
-<signal name="N$14">
+<signal name="P1.13">
 <contactref element="BTN1" pad="1" route="any" routetag="G$1.P"/>
 <contactref element="BTN1" pad="2" route="any" routetag="G$1.P"/>
